Commit message: Temp commit for ros2_control on real robot

File: description/gazebo_control.xacro (robot description, xacro)
@@ -6,6 +6,6 @@
             <left_joint>left_wheel_joint</left_joint>
             <right_joint>right_wheel_joint</right_joint>
-            <wheel_separation>0.35</wheel_separation>
-            <wheel_diameter>0.1</wheel_diameter>
+            <wheel_separation>0.194</wheel_separation>
+            <wheel_diameter>0.064</wheel_diameter>
             <!-- Limits -->
             <max_wheel_torque>200</max_wheel_torque>

File: description/lidar.xacro (robot description, xacro)
@@ -2,10 +2,10 @@
 <robot xmlns:xacro="http://www.ros.org/wiki/xacro" >
     <joint name="laser_joint" type="fixed">
-        <origin xyz="0.1 0.0 0.175" rpy="0.0 0.0 0.0"/>
+        <origin xyz="0.15 0.0 0.131" rpy="0.0 0.0 0.0"/>
         <parent link="chassis"/>
         <child link="laser_frame"/>
     </joint>
     <link name="laser_frame">
-        <xacro:inertial_cylinder mass="0.1" radius="0.05" length="0.04">
+        <xacro:inertial_cylinder mass="0.1" radius="0.035" length="0.025">
             <origin xyz="0 0 0"  rpy="0 0 0"/>
         </xacro:inertial_cylinder>
@@ -13,5 +13,5 @@
             <origin xyz="0.0 0.0 0.0" rpy="0.0 0.0 0.0"/>
             <geometry>
-                <cylinder radius="0.05" length="0.04"/>
+                <cylinder radius="0.035" length="0.025"/>
             </geometry>
             <material name="">
@@ -30,5 +30,5 @@
         <material>Gazebo/Red</material>
         <sensor name="laser" type="ray">
-            <pose> 0 0 0 0 0 0 </pose>
+            <pose> 0 0 0 0 0 pi </pose>
             <visualize>true</visualize>
             <update_rate>10</update_rate>
@@ -36,13 +36,18 @@
                 <scan>
                     <horizontal>
-                        <samples>360</samples>
-                        <min_angle>-3.14</min_angle>
-                        <max_angle>3.14</max_angle>
+                        <samples>1200</samples>
+                        <min_angle>6.283</min_angle>
+                        <max_angle>0</max_angle>
                     </horizontal>
                 </scan>
                 <range>
                     <min>0.3</min>
-                    <max>12</max>
+                    <max>24</max>
                 </range>
+                <noise>
+                    <type>gaussian</type> <!-- Тип шума -->
+                    <mean>0.0</mean> <!-- Среднее значение шума -->
+                    <stddev>0.10</stddev> <!-- Стандартное отклонение -->
+                </noise>
             </ray>
             <plugin name="laser_controller" filename="libgazebo_ros_ray_sensor.so">

File: description/robot_core.xacro (robot description, xacro)
@@ -9,10 +9,10 @@
     <xacro:property name="wheel_thickness" value="0.011"/>
     <xacro:property name="wheel_mass" value="0.05"/>
-    <xacro:property name="wheel_offset_x" value="0.226"/>
-    <xacro:property name="wheel_offset_y" value="0.166"/>
+    <xacro:property name="wheel_offset_x" value="0.154"/>
+    <xacro:property name="wheel_offset_y" value="0.097"/>
     <xacro:property name="wheel_offset_z" value="0.01"/>
     <xacro:property name="caster_wheel_radius" value="0.01"/>
     <xacro:property name="caster_wheel_mass" value="0.01"/>
-    <xacro:property name="caster_wheel_offset_x" value="0.075"/>
+    <xacro:property name="caster_wheel_offset_x" value="0.017"/>
     <xacro:property name="caster_wheel_offset_z" value="${wheel_offset_z - wheel_radius + caster_wheel_radius}"/>
     <material name="white">
@@ -33,4 +33,12 @@
     <!-- BASE LINK -->
     <link name="base_link">
+    </link>
+    <!-- BASE_FOOTPRINT LINK -->
+    <joint name="base_footprint_joint" type="fixed">
+        <parent link="base_link"/>
+        <child link="base_footprint"/>
+        <origin xyz="0 0 0" rpy="0 0 0"/>
+    </joint>
+    <link name="base_footprint">
     </link>
     <!-- CHASSIS LINK -->
@@ -86,4 +94,5 @@
     <gazebo reference="left_wheel">
         <material>Gazebo/Blue</material>
+        <mu1 value = "0.1"/>
     </gazebo>
     <!-- RIGHT WHEEL LINK -->
@@ -112,4 +121,5 @@
     <gazebo reference="right_wheel">
         <material>Gazebo/Blue</material>
+        <mu1 value = "0.1"/>
     </gazebo>
     <!-- CASTER WHEEL LINK -->
